File: kicad/st_amplifier/st_amplifier.kicad_pcb (KiCad board)
At the start: 2 copper layers, 0 parts

Commit message: New commit.
Parts:
- added C1: 470мк 50В, CAPACITOR_CD263_5.08_D10, F.Cu at (160.0, 40.6)
- added C11: 100мк 50В, CAPACITOR_5.08_D13, F.Cu at (137.2, 26.7)
- added C12: 10 п, CAPACITOR_K10-17, F.Cu at (26.7, 96.5)
- added C13: 10 п, CAPACITOR_K10-17, F.Cu at (55.9, 96.5)
- added C14: 2200мк 50В, CAPACITOR_10_D22, F.Cu at (188.0, 63.5)
- added C16: 2200мк 50В, CAPACITOR_10_D22, F.Cu at (160.0, 63.5)
- added C2: 22мк 35В, CAPACITOR_CD263_2.54_D6.3, F.Cu at (186.7, 26.7)
- added C20: 2.2 мк, CAPACITOR_CBB21_20_24x11, F.Cu at (172.7, 105.4)
- added C21: 100 п, CAPACITOR_K10-17, F.Cu at (41.9, 96.5)
- added C22: 0.1 мк, CAPACITOR_K10-17, F.Cu at (55.9, 82.5)
- added C23: 0.1 мк, CAPACITOR_K10-17, F.Cu at (26.7, 90.2)
- added C24: 2.2 мк, CAPACITOR_CBB21_20_24x11, F.Cu at (141.0, 105.4)
- added C25: 100мк 50В, CAPACITOR_5.08_D13, F.Cu at (137.2, 44.5)
- added C26: 2.2 мк, CAPACITOR_CBB21_20_24x11, F.Cu at (172.7, 86.4)
- added C27: 100 п, CAPACITOR_K10-17, F.Cu at (26.7, 104.1)
- added C28: 0.1 мк, CAPACITOR_K10-17, F.Cu at (55.9, 90.2)
- added C3: 0.1 мк, CAPACITOR_K10-17, F.Cu at (41.9, 82.5)
- added C30: 100мк 50В, CAPACITOR_5.08_D13, F.Cu at (118.1, 44.5)
- added C31: 470мк 50В, CAPACITOR_CD263_5.08_D10, F.Cu at (172.7, 40.6)
- added C33: 470мк 50В, CAPACITOR_CD263_5.08_D10, F.Cu at (160.0, 26.7)
- added C4: 470мк 50В, CAPACITOR_CD263_5.08_D10, F.Cu at (172.7, 26.7)
- added C5: 22мк 35В, CAPACITOR_CD263_2.54_D6.3, F.Cu at (186.7, 40.6)
- added C6: 0.1 мк, CAPACITOR_K10-17, F.Cu at (26.7, 82.5)
- added C7: 100мк 50В, CAPACITOR_5.08_D13, F.Cu at (119.4, 26.7)
- added C8: 2.2 мк, CAPACITOR_CBB21_20_24x11, F.Cu at (141.0, 86.4)
- added C9: 0.1 мк, CAPACITOR_K10-17, F.Cu at (41.9, 90.2)
- added DA1: LM7815, TO220_VERT_POZ, F.Cu at (31.8, 39.4)
- added DA2: LM7915, TO220_VERT_POZ, F.Cu at (21.6, 39.4)
- added DA3: LME49720MA, SOIC8, F.Cu at (69.8, 24.1)
- added DA4: TDA7293, MULTIWATT15, F.Cu at (67.3, 62.2)
- added DA5: TDA7293, MULTIWATT15, F.Cu at (102.9, 62.2)
- added VD1: 1N4007, DO-41, F.Cu at (90.2, 45.7)
- added XS1: DG126-5.0-03P-14, DG126-5.0-03P-14, F.Cu at (52.1, 43.2)
- added XS2: WF-4, WF-4, F.Cu at (34.3, 58.4)
- added XS3: DG126-5.0-02P-14, DG126-5.0-02P-14, F.Cu at (53.3, 26.7)
- added XS4: WF-2, WF-2, F.Cu at (45.7, 58.4)
- added XS5: WF-2, WF-2, F.Cu at (22.9, 58.4)
- added XS6: DG126-5.0-02P-14, DG126-5.0-02P-14, F.Cu at (72.4, 44.5)

Commit message: New commit.
Parts:
- added C10: 1 мк, CAPACITOR_CBB21_15_16x6, F.Cu at (213.4, 74.9)
- added C15: 1 мк, CAPACITOR_CBB21_15_16x6, F.Cu at (213.4, 54.6)
- added C17: 1 мк, CAPACITOR_CBB21_15_16x6, F.Cu at (213.4, 44.5)
- added C18: 10мк 50В, CAPACITOR_0511, F.Cu at (71.1, 100.3)
- added C19: 10мк 50В, CAPACITOR_0511, F.Cu at (71.1, 91.4)
- added C29: 1 мк, CAPACITOR_CBB21_15_16x6, F.Cu at (213.4, 24.1)
- added C32: 1 мк, CAPACITOR_CBB21_15_16x6, F.Cu at (213.4, 34.3)
- added C34: 1 мк, CAPACITOR_CBB21_15_16x6, F.Cu at (213.4, 64.8)
- added L1: 0,7 мкГн, RESISTOR_2W, F.Cu at (101.6, 87.6)
- added L2: 0,7 мкГн, RESISTOR_2W, F.Cu at (101.6, 100.3)
- added R1: 1 к +/-0.5%, RESISTOR_1W, F.Cu at (240.0, 83.8)
- added R10: 22 к, RESISTOR_0.25W, F.Cu at (269.2, 72.4)
- added R11: 1 к, RESISTOR_0.25W, F.Cu at (269.2, 40.6)
- added R12: 22 к, RESISTOR_0.25W, F.Cu at (269.2, 53.3)
- added R13: 1 к +/- 0.5%, RESISTOR_1W, F.Cu at (240.0, 66.0)
- added R14: 2 к +/- 0.5%, RESISTOR_1W, F.Cu at (240.0, 55.9)
- added R15: 12 к +/-0.5%, RESISTOR_1W, F.Cu at (240.0, 45.7)
- added R16: 12 к +/-0.5%, RESISTOR_1W, F.Cu at (240.0, 74.9)
- added R17: 10, RESISTOR_2W, F.Cu at (210.8, 99.1)
- added R18: 22 к, RESISTOR_0.25W, F.Cu at (269.2, 47.0)
- added R19: 2,7 к, RESISTOR_0.25W, F.Cu at (269.2, 26.7)
- added R2: 2 к +/-0.5%, RESISTOR_1W, F.Cu at (240.0, 25.4)
- added R20: 10, RESISTOR_2W, F.Cu at (210.8, 121.9)
- added R3: 10, RESISTOR_2W, F.Cu at (212.1, 110.5)
- added R4: 2,7 к, RESISTOR_0.25W, F.Cu at (269.2, 34.3)
- added R5: 10, RESISTOR_2W, F.Cu at (210.8, 87.6)
- added R6: 47 к +/-0.5%, RESISTOR_1W, F.Cu at (240.0, 94.0)
- added R7: 5.1 к, RESISTOR_0.25W, F.Cu at (269.2, 59.7)
- added R8: 47 к +/-0.5%, RESISTOR_1W, F.Cu at (240.0, 35.6)
- added R9: 22 к, RESISTOR_0.25W, F.Cu at (269.2, 66.0)
