File: kicad/st_amplifier/st_amplifier.sch (KiCad schematic (older format))
At the start: 67 parts

Commit message: Fixed errors.
Parts:
- R1: value 1 к +/-0.5% -> 2 к +/-0.5%
- R13: value 1 к +/- 0.5% -> 2 к +/-0.5%
- R14: value 2 к +/- 0.5% -> 28.7 к +/-0.5%
- R19, R4: value 2,7 к -> 100
- R2: value 2 к +/-0.5% -> 28.7 к +/-0.5%
- R6, R8: value 47 к +/-0.5% -> 22.1 к +/-0.5%
Connections:
- net +15V: now also C23.1, DA3.8 (V+); no longer C22.1, DA3.4 (V-)
- net -15V: now also C22.1, DA3.4 (V-); no longer C23.1, DA3.8 (V+)
- net -29V: now also C16.2, C33.2; no longer C16.1, C33.1
- net GND: now also C16.1, C33.1; no longer C16.2, C33.2
Changed lines of the file:
@@
 Sheet 1 1
 Title ""
-Date "3 may 2015"
+Date "22 may 2015"
 Rev ""
 Comp ""
@@
 	13050 3250 12800 3250
 Wire Wire Line
-	12800 3650 12800 3250
+	12800 3250 12800 3650
 Connection ~ 9750 4050
 Wire Wire Line
@@
 	12700 3850 12700 3950
 Wire Wire Line
-	11450 3850 12700 3850
-Wire Wire Line
 	12000 4750 12700 4750
 Wire Wire Line
@@
 	11850 4850 11850 4750
 Wire Wire Line
-	11550 4750 11850 4750
+	11850 4750 11550 4750
 Connection ~ 11550 4550
 Wire Wire Line
@@
 	9100 3450 9100 3750
 Connection ~ 9100 3550
-Wire Wire Line
-	12200 3850 12200 3850
 Wire Wire Line
 	12400 3950 12400 3850
@@
 P 9300 3100
 F 0 "R1" H 9450 3350 71  0000 C CNN
-F 1 "1 к  +/-0.5%" H 9450 3250 71  0000 C CNN
+F 1 "2 к  +/-0.5%" H 9450 3250 71  0000 C CNN
 F 2 "" H 9300 3100 60  0001 C CNN
 F 3 "" H 9300 3100 60  0001 C CNN
@@
 P 10500 3100
 F 0 "R2" H 10650 3350 71  0000 C CNN
-F 1 "2 к  +/-0.5%" H 10650 3250 71  0000 C CNN
+F 1 "28.7 к  +/-0.5%" H 10650 3250 71  0000 C CNN
 F 2 "" H 10500 3100 60  0001 C CNN
 F 3 "" H 10500 3100 60  0001 C CNN
@@
 L CAPITORS_ELECTROLYTIC C16
 U 1 1 532EE840
-P 12400 5250
-F 0 "C16" V 12500 4800 71  0000 C CNN
-F 1 "2200мк 50В" V 12600 4800 71  0000 C CNN
-F 2 "" H 12400 5250 60  0001 C CNN
-F 3 "" H 12400 5250 60  0001 C CNN
-	1    12400 5250
-	0    1    1    0
+P 12400 5500
+F 0 "C16" V 12600 5050 71  0000 C CNN
+F 1 "2200мк 50В" V 12500 5050 71  0000 C CNN
+F 2 "" H 12400 5500 60  0001 C CNN
+F 3 "" H 12400 5500 60  0001 C CNN
+	1    12400 5500
+	0    1    -1   0
 $EndComp
 $Comp
@@
 	12850 6800 12600 6800
 Wire Wire Line
-	12600 7200 12600 6800
+	12600 6800 12600 7200
 Connection ~ 9550 7600
 Wire Wire Line
@@
 	11650 8400 11650 8300
 Wire Wire Line
-	11350 8300 11650 8300
+	11650 8300 11350 8300
 Connection ~ 11350 8100
 Wire Wire Line
@@
 P 9100 6650
 F 0 "R13" H 9250 6900 71  0000 C CNN
-F 1 "1 к +/- 0.5%" H 9250 6800 71  0000 C CNN
+F 1 "2 к +/-0.5%" H 9250 6800 71  0000 C CNN
 F 2 "" H 9100 6650 60  0001 C CNN
 F 3 "" H 9100 6650 60  0001 C CNN
@@
 P 10300 6650
 F 0 "R14" H 10450 6900 71  0000 C CNN
-F 1 "2 к +/- 0.5%" H 10450 6800 71  0000 C CNN
+F 1 "28.7 к +/-0.5%" H 10450 6800 71  0000 C CNN
 F 2 "" H 10300 6650 60  0001 C CNN
 F 3 "" H 10300 6650 60  0001 C CNN
@@
 L CAPITORS_ELECTROLYTIC C33
 U 1 1 552A86CA
-P 12200 8800
-F 0 "C33" V 12300 8350 71  0000 C CNN
-F 1 "2200мк 50В" V 12400 8350 71  0000 C CNN
-F 2 "" H 12200 8800 60  0001 C CNN
-F 3 "" H 12200 8800 60  0001 C CNN
-	1    12200 8800
-	0    1    1    0
+P 12200 9050
+F 0 "C33" V 12350 8600 71  0000 C CNN
+F 1 "2200мк 50В" V 12250 8600 71  0000 C CNN
+F 2 "" H 12200 9050 60  0001 C CNN
+F 3 "" H 12200 9050 60  0001 C CNN
+	1    12200 9050
+	0    1    -1   0
 $EndComp
 $Comp
@@
 P 6100 5150
 F 0 "R8" H 6750 5250 71  0000 C CNN
-F 1 "47 к +/-0.5%" H 7000 5100 71  0000 C CNN
+F 1 "22.1 к +/-0.5%" H 7050 5100 71  0000 C CNN
 F 2 "" H 6100 5150 60  0001 C CNN
 F 3 "" H 6100 5150 60  0001 C CNN
@@
 P 4850 4750
 F 0 "R6" H 4950 4600 71  0000 C CNN
-F 1 "47 к +/-0.5%" H 5200 4450 71  0000 C CNN
+F 1 "22.1 к +/-0.5%" H 5250 4450 71  0000 C CNN
 F 2 "" H 4850 4750 60  0001 C CNN
 F 3 "" H 4850 4750 60  0001 C CNN
@@
 P 9300 3850
 F 0 "R4" H 9450 4100 71  0000 C CNN
-F 1 "2,7 к" H 9450 4000 71  0000 C CNN
+F 1 "100" H 9450 4000 71  0000 C CNN
 F 2 "" H 9300 3850 60  0001 C CNN
 F 3 "" H 9300 3850 60  0001 C CNN
@@
 P 9100 7400
 F 0 "R19" H 9250 7650 71  0000 C CNN
-F 1 "2,7 к" H 9250 7550 71  0000 C CNN
+F 1 "100" H 9250 7550 71  0000 C CNN
 F 2 "" H 9100 7400 60  0001 C CNN
 F 3 "" H 9100 7400 60  0001 C CNN
@@
 Wire Wire Line
 	6350 6350 7150 6350
+Text Label 7150 6150 2    60   ~ 0
+-15V
 Text Label 7150 6350 2    60   ~ 0
--15V
-Text Label 7150 6150 2    60   ~ 0
 +15V
 $Comp
@@
 Text Label 2450 2600 2    60   ~ 0
 CLIP_2
+Wire Wire Line
+	11450 3850 12700 3850
 $EndSCHEMATC
