File: kicad/2-way_active_filter/2-way_active_filter.sch (KiCad schematic (older format))
At the start: 64 parts

Commit message: Adding new shema for 2 way active filter.
Parts:
- removed C16, C9: 220 п, symbol CAPITORS
- removed C21, C22: 0.1 мк, symbol CAPITORS
- removed R17: 10, symbol RESISTOR
- added C1, C2, C32, C33: 2.2 мк, symbol CAPITORS
- added C12, C8: 0.1 мк, symbol CAPITORS
- added C14, C15, C20, C30, C31: 22 п, symbol CAPITORS
- added C34, C35, C4, C5, C6: 220 п, symbol CAPITORS
- added unit 3 of DA3
- added unit 2 of DA3
- added DA4: LME49740MA, ~, symbol LME49740
- added FU1: 0.1 А, ~, symbol PROTECTOR
- added R1, R2: 22 к, symbol RESISTOR
- added R10, R11, R12, R13, R14, R9: 10 к, symbol RESISTOR
- added R38, R39, R40, R41, R8: 10, symbol RESISTOR
- added R5, R6: 220, symbol RESISTOR
- added XS2: WF-4, ~, symbol PIN_M_4
- added XS3: WF-3, ~, symbol PIN_M_3
- added XS5: WF-5, ~, symbol PIN_M_5
- added XS6, XS9: PLS-3, ~, symbol PIN_M_3
- added XS7, XS8: PLS-2, ~, symbol PIN_M_2
- C10: renamed from C4; value 4700мк 25В -> 4700мк 35В
- C9: renamed from C1; value 4700мк 25В -> 4700мк 35В
- DA3, DA5: value LME49720MA -> LME49740MA; symbol LME49720 -> LME49740
- DA5: renamed from DA4; value LME49720MA -> LME49740MA; symbol LME49720 -> LME49740
- R17: renamed from R1; value 10 к -> 30 к
- R26: renamed from R11; value 30 к -> 1 к
- R36: renamed from R6; value 10 к -> 50 к
- R37: renamed from R18; value 10 к -> 50 к
- TV1: value BVEI 481 1120 -> BVEI 481 0120
- XS10: renamed from XS2; value WF-3 -> WF-4; symbol PIN_M_3 -> PIN_M_4
- XS11: renamed from XS4; value WF-3 -> WF-4; symbol PIN_M_3 -> PIN_M_4
- renumbered C14 to C11, C15 to C13, C2 to C16, C5 to C17, C3 to C18, C6 to C19, C23 to C21, C17 to C22, C19 to C23, C11 to C24, C8 to C25, C12 to C26, C13 to C27, C18 to C28, C20 to C29, C7 to C3, C10 to C7, R12 to R15, R19 to R16, R20 to R18, R27 to R19, R21 to R20, R22 to R21, R7 to R22, R3 to R23, R8 to R24, R2 to R25, R13 to R27, R23 to R28, R24 to R29, R10 to R3, R25 to R30, R9 to R31, R26 to R32, R14 to R33, R15 to R34, R16 to R35, R5 to R7, VD3 to VD2, VD2 to VD3, XS3 to XS1, XS1 to XS4
Connections:
- wire segments 179 -> 287
Other:
- note added: "B+"
- note added: "B-"
- note added: "БАЛАНСНЫЙ\n ВХОД"
- note added: "Выбор конденсаторов:\n\nC22 = C23 = C24 = C25 = C28 = C29 = C\n\nf = 60 - 600 Гц, C = 0.047 мкФ\nf = 600 - 6 000 Гц, C = 0.0047 мкФ\nf = 4000 - 20 000 Гц, C = 0.001 мкФ"
- note added: "ЛИНЕЙНЫЙ\n ВХОД"
- note added: "ЛИНЕЙНЫЙ\n ВЫХОД"
- note added: "Расчёт фазового фильтра 4-го порядка:\n\nR22 + R24 = R26 + R27 = R\nR23 = 4 * R25\nC22 = C23 = C\n\nR = 1 / 2 *PI * SQRT(2) * f * C"
- note added: "Расчёт фильтра Бесселя 4-го порядка:\n\nR16 + R18 = R20 + R21 = R1\nR28 + R29 = R30 + R32 = R2\nC24 = C25 = C28 = C29 = C\n\nR1 = 1 / 2 *PI * SQRT(2) * 0.8918 * f * C\nR2 = 1 / 2 *PI * SQRT(2) * f * C"
- note added: "ФАЗОВЫЙ ФИЛЬТР 4-ГО ПОРЯДКА"
- note added: "ФИЛЬТР БЕССЕЛЯ 4-ПОРЯДКА"
- note removed: "ВХОД"
- note removed: "Расчёт фазового фильтра 4-го порядка:\n\nR7+R8 = R11 + R13 = R\nR3 = 4 * R2\nC7 = C8 = C\n\nR = 1 / 2 *PI * SQRT(2) * f * C"
- note removed: "Расчёт фильтра Бесселя 4-го порядка:\n\nR19 + R20 = R21 + R22 = R1\nR23 + R24 = R25 + R26 = R2\nC15 = C16 = C17 = C18 = C\n\nR1 = 1 / 2 *PI * SQRT(2) * 0.8918 * f * C\nR2 = 1 / 2 *PI * SQRT(2) * f * C"
- note removed: "ФАЗОВЫЙ ФИЛЬТР 4-ГО ПОРЯДКА\n настраивается на 100 - 1000 Гц"
- note removed: "ФИЛЬТР БЕССЕЛЯ 4-ПОРЯДКА \nнастраивается на 100 - 1000 Гц"
- moved on the sheet: C10, C11, C13, C16, C17, C18, C19, C21, C22, C23, C24, C25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

Commit message: Adding new version st_amplifier (rev. 1).
Parts:
- added C36, C37, C40, C41: 0.1 мк, symbol CAPITORS
- added C38, C39: 220 п, symbol CAPITORS
- added DA7: LME49720MA, ~, symbol LME49720
- added R42: 0, symbol RESISTOR
- added R43, R44, R45, R46: 10, symbol RESISTOR
- added XS12: WF-4, ~, symbol PIN_M_4
- DA3: value LME49740MA -> LME49720MA; symbol LME49740 -> LME49720
- DA4: renamed from DA3; value LME49740MA -> LME49720MA; symbol LME49740 -> LME49720
- renumbered DA4 to DA6
Connections:
- wire segments 287 -> 330
Other:
- note added: "* Перемычка устанавливается если нужен\n только один линейный вход"
- note added: "БАЛАНСНЫЙ\n ВЫХОД"
- moved on the sheet: C1, C10, C11, C12, C13, C14, C15, C16, C17, C18, C19, C2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

Commit message: New commit.
Parts:
- added C42, C43, C44: 22 п, symbol CAPITORS
- added R47, R48, R51, R52: 10 к, symbol RESISTOR
- added R49, R50: 50 к, symbol RESISTOR_TRIMMING
- added R53, R54: 30 к, symbol RESISTOR
- added R55, R56, R57, R58, R59, R60, R61, R62, R63, R64: 4.7, symbol RESISTOR
- added XS13, XS14, XS15: DG126-5.0-03P-14, ~, symbol PIN_F_3
- DA1: value LM7815 -> L7815CV
- DA2: value LM7915 -> L7915CV
- R14: value 10 к -> 30 к
- TV1: symbol BVEI_302_2028 -> BVEI_481_0120
Connections:
- wire segments 330 -> 375
Other:
- note added: "*"
- note added: "* Перемычка устанавливается если нужен\n только один линейный вход, в этом случае\n DA3 не впаивается"
- note added: "**"
- note added: "** Если усиление входного сигнала\n не нужно то C20 и R13 не впаивать,\n а в место R14 впаять перемыку"
- note removed: "* Перемычка устанавливается если нужен\n только один линейный вход"
- moved on the sheet: C11, C12, C13, C15, C27, C36, C37, C38, C39, C4, C40, C41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

Commit message: 2-way active filter.
Parts:
- removed XS15: DG126-5.0-03P-14, ~, symbol PIN_F_3
- XP3: renamed from XS5; value WF-5 -> WF-6; symbol PIN_M_5 -> PIN_M_6
- renumbered XS1 to XP1, XS2 to XP10, XS12 to XP11, XS3 to XP2, XS6 to XP4, XS7 to XP5, XS8 to XP6, XS9 to XP7, XS10 to XP8, XS4 to XS1, XS13 to XS2, XS14 to XS3, XS11 to XS9
Connections:
- wire segments 375 -> 372
Other:
- moved on the sheet: XS2, XS3
Changed lines of the file:
@@
 Sheet 1 1
 Title ""
-Date "9 jul 2015"
+Date "19 jul 2015"
 Rev ""
 Comp ""
@@
 Text Label 4300 4200 2    60   ~ 0
 GND
-Text Label 12100 1850 2    60   ~ 0
+Text Label 12250 1850 2    60   ~ 0
 -15V
-Text Label 12100 1750 2    60   ~ 0
+Text Label 12250 1750 2    60   ~ 0
 GND
 $Comp
@@
 AR Path="/52F0D059" Ref="XS?"  Part="1"
 AR Path="/52F0D221" Ref="XS?"  Part="1"
-AR Path="/5303196E" Ref="XS4"  Part="1"
-F 0 "XS4" H 4200 1900 50  0000 L BNN
+AR Path="/5303196E" Ref="XS1"  Part="1"
+F 0 "XS1" H 4200 1900 50  0000 L BNN
 F 1 "DG126-5.0-02P-14" H 3900 1800 50  0000 L BNN
 F 2 "~" H 4500 1850 50  0001 C CNN
@@
 	0    1    1    0
 $EndComp
-Text Label 12100 1650 2    60   ~ 0
+Text Label 12250 1650 2    60   ~ 0
 +15V
 $Comp
-L PIN_M_3 XS1
+L PIN_M_3 XP1
 U 1 1 557D49EA
 P 4000 4100
-F 0 "XS1" H 4100 4300 50  0000 L BNN
+F 0 "XP1" H 4100 4300 50  0000 L BNN
 F 1 "WF-3" H 4050 4200 50  0000 L BNN
 F 2 "~" H 4450 4250 50  0001 C CNN
@@
 P 20400 4000
 AR Path="/530320C3" Ref="XS?"  Part="1"
-AR Path="/557DEBAD" Ref="XS10"  Part="1"
-F 0 "XS10" H 20450 4200 50  0000 L BNN
+AR Path="/557DEBAD" Ref="XP8"  Part="1"
+F 0 "XP8" H 20450 4200 50  0000 L BNN
 F 1 "WF-4" H 20450 4100 50  0000 L BNN
 F 2 "~" H 20850 4150 50  0001 C CNN
@@
 P 20400 5400
 AR Path="/530320C3" Ref="XS?"  Part="1"
-AR Path="/557DF38E" Ref="XS11"  Part="1"
-F 0 "XS11" H 20450 5600 50  0000 L BNN
+AR Path="/557DF38E" Ref="XS9"  Part="1"
+F 0 "XS9" H 20450 5600 50  0000 L BNN
 F 1 "WF-4" H 20450 5500 50  0000 L BNN
 F 2 "~" H 20850 5550 50  0001 C CNN
@@
 $EndComp
 $Comp
-L PIN_M_3 XS9
+L PIN_M_3 XP7
 U 1 1 55892DD8
 P 15600 6350
-F 0 "XS9" V 15850 6500 50  0000 L BNN
+F 0 "XP7" V 15850 6500 50  0000 L BNN
 F 1 "PLS-3" V 15950 6450 50  0000 L BNN
 F 2 "~" H 16050 6500 50  0001 C CNN
@@
 $EndComp
 $Comp
-L PIN_M_3 XS6
+L PIN_M_3 XP4
 U 1 1 55892DE3
 P 11900 6350
-F 0 "XS6" V 12100 6500 50  0000 L BNN
+F 0 "XP4" V 12100 6500 50  0000 L BNN
 F 1 "PLS-3" V 12200 6450 50  0000 L BNN
 F 2 "~" H 12350 6500 50  0001 C CNN
@@
 $EndComp
 $Comp
-L PIN_M_2 XS7
+L PIN_M_2 XP5
 U 1 1 5589343C
 P 12950 4600
-F 0 "XS7" V 13150 4750 50  0000 L BNN
+F 0 "XP5" V 13150 4750 50  0000 L BNN
 F 1 "PLS-2" V 13250 4700 50  0000 L BNN
 F 2 "~" H 13400 4750 50  0001 C CNN
@@
 $EndComp
 $Comp
-L PIN_M_2 XS8
+L PIN_M_2 XP6
 U 1 1 5589367A
 P 14150 5250
-F 0 "XS8" H 14650 5200 50  0000 L BNN
+F 0 "XP6" H 14650 5200 50  0000 L BNN
 F 1 "PLS-2" H 14600 5100 50  0000 L BNN
 F 2 "~" H 14600 5400 50  0001 C CNN
@@
 $EndComp
 $Comp
-L PIN_M_3 XS3
+L PIN_M_3 XP2
 U 1 1 55895583
 P 4000 8250
-F 0 "XS3" H 4200 8450 50  0000 L BNN
+F 0 "XP2" H 4200 8450 50  0000 L BNN
 F 1 "WF-3" H 4150 8350 50  0000 L BNN
 F 2 "~" H 4450 8400 50  0001 C CNN
@@
 P 20400 7950
 AR Path="/530320C3" Ref="XS?"  Part="1"
-AR Path="/558BCB0D" Ref="XS2"  Part="1"
-F 0 "XS2" H 20500 8150 50  0000 L BNN
+AR Path="/558BCB0D" Ref="XP10"  Part="1"
+F 0 "XP10" H 20500 8150 50  0000 L BNN
 F 1 "WF-4" H 20450 8050 50  0000 L BNN
 F 2 "~" H 20850 8100 50  0001 C CNN
@@
 $EndComp
 $Comp
-L PIN_M_5 XS5
+L PIN_M_6 XP3
 U 1 1 558BD5F7
 P 7900 3750
-F 0 "XS5" V 8500 3500 50  0000 L BNN
-F 1 "WF-5" V 8400 3450 50  0000 L BNN
+F 0 "XP3" V 8500 3450 50  0000 L BNN
+F 1 "WF-6" V 8400 3400 50  0000 L BNN
 F 2 "~" H 8350 3900 50  0001 C CNN
 F 3 "" H 7900 3750 60  0001 C CNN
@@
 	0    -1   -1   0
 $EndComp
-Text Label 8300 3950 1    60   ~ 0
+Text Label 8400 3950 1    60   ~ 0
 GND
 Text Label 10100 5450 1    60   ~ 0
@@
 P 20400 10250
 AR Path="/530320C3" Ref="XS?"  Part="1"
-AR Path="/55912278" Ref="XS12"  Part="1"
-F 0 "XS12" H 20600 10450 50  0000 L BNN
+AR Path="/55912278" Ref="XP11"  Part="1"
+F 0 "XP11" H 20600 10450 50  0000 L BNN
 F 1 "WF-4" H 20600 10350 50  0000 L BNN
 F 2 "~" H 20850 10400 50  0001 C CNN
@@
 	8500 2350 9950 2350
 Connection ~ 9350 1150
-Wire Wire Line
-	8500 1150 10350 1150
 Connection ~ 7000 1150
 Wire Wire Line
@@
 Connection ~ 19050 7950
 Wire Wire Line
-	7900 3750 7900 6500
-Wire Wire Line
-	8000 6700 8000 3750
-Wire Wire Line
 	4000 8350 4350 8350
 Wire Wire Line
@@
 	10000 4600 10300 4600
 Wire Wire Line
-	8200 3750 8200 4100
-Wire Wire Line
-	8200 4100 8550 4100
+	8300 3750 8300 4100
 Wire Wire Line
 	6900 4100 7900 4100
-Connection ~ 7900 4100
 Wire Wire Line
 	5250 3550 6050 3550
@@
 Wire Wire Line
 	10150 7800 10850 7800
-Wire Wire Line
-	10850 6700 8000 6700
 Connection ~ 10850 7500
 Wire Wire Line
@@
 Connection ~ 17250 11250
 Connection ~ 18900 11050
-Wire Wire Line
-	8100 3750 8100 6600
-Wire Wire Line
-	8100 6600 10950 6600
 Wire Wire Line
 	18900 11900 18200 11900
@@
 Text Notes 20900 10400 0    60   ~ 0
 БАЛАНСНЫЙ\n   ВЫХОД
-Wire Wire Line
-	7900 6500 11050 6500
 Text Notes 20900 8100 0    60   ~ 0
 ЛИНЕЙНЫЙ\n  ВЫХОД
@@
 $EndComp
 Wire Wire Line
-	8300 3950 8300 3750
+	8400 3950 8400 3750
 Wire Wire Line
 	10550 4400 10800 4400
@@
 L PIN_F_3 XS?
 U 1 1 559E39B2
+P 11900 1650
+AR Path="/52F0D059" Ref="XS?"  Part="1"
+AR Path="/52F0D221" Ref="XS?"  Part="1"
+AR Path="/559E39B2" Ref="XS3"  Part="1"
+F 0 "XS3" H 12050 1850 50  0000 L BNN
+F 1 "DG126-5.0-03P-14" H 11750 1750 50  0000 L BNN
+F 2 "~" H 12350 1800 50  0001 C CNN
+F 3 "" H 11900 1650 60  0001 C CNN
+	1    11900 1650
+	-1   0    0    -1
+$EndComp
+Wire Wire Line
+	9950 1150 9950 1650
+Wire Wire Line
+	9950 1650 10350 1650
+Wire Wire Line
+	9950 1850 10350 1850
+Wire Wire Line
+	9950 2350 9950 1850
+$Comp
+L PIN_F_3 XS?
+U 1 1 559E3EAF
 P 10350 1650
 AR Path="/52F0D059" Ref="XS?"  Part="1"
 AR Path="/52F0D221" Ref="XS?"  Part="1"
-AR Path="/559E39B2" Ref="XS14"  Part="1"
-F 0 "XS14" H 10500 1850 50  0000 L BNN
+AR Path="/559E3EAF" Ref="XS2"  Part="1"
+F 0 "XS2" H 10500 1850 50  0000 L BNN
 F 1 "DG126-5.0-03P-14" H 10200 1750 50  0000 L BNN
 F 2 "~" H 10800 1800 50  0001 C CNN
@@
 $EndComp
 Wire Wire Line
-	9950 1150 9950 1650
-Wire Wire Line
-	9950 1650 10350 1650
-Wire Wire Line
-	9950 1850 10350 1850
-Wire Wire Line
-	9950 2350 9950 1850
-$Comp
-L PIN_F_3 XS?
-U 1 1 559E3E9B
-P 11750 1650
-AR Path="/52F0D059" Ref="XS?"  Part="1"
-AR Path="/52F0D221" Ref="XS?"  Part="1"
-AR Path="/559E3E9B" Ref="XS15"  Part="1"
-F 0 "XS15" H 11900 1850 50  0000 L BNN
-F 1 "DG126-5.0-03P-14" H 11600 1750 50  0000 L BNN
-F 2 "~" H 12200 1800 50  0001 C CNN
-F 3 "" H 11750 1650 60  0001 C CNN
-	1    11750 1650
-	-1   0    0    -1
-$EndComp
-$Comp
-L PIN_F_3 XS?
-U 1 1 559E3EAF
-P 10350 1150
-AR Path="/52F0D059" Ref="XS?"  Part="1"
-AR Path="/52F0D221" Ref="XS?"  Part="1"
-AR Path="/559E3EAF" Ref="XS13"  Part="1"
-F 0 "XS13" H 10500 1350 50  0000 L BNN
-F 1 "DG126-5.0-03P-14" H 10200 1250 50  0000 L BNN
-F 2 "~" H 10800 1300 50  0001 C CNN
-F 3 "" H 10350 1150 60  0001 C CNN
-	1    10350 1150
-	1    0    0    -1
-$EndComp
-Connection ~ 9950 1150
-Wire Wire Line
-	10350 1250 10050 1250
-Wire Wire Line
-	10350 1350 10150 1350
-Wire Wire Line
-	10150 1350 10150 1850
-Connection ~ 10150 1850
-Wire Wire Line
-	11750 1650 12100 1650
-Wire Wire Line
-	12100 1750 11750 1750
-Wire Wire Line
-	12100 1850 11750 1850
-Wire Wire Line
-	10050 1250 10050 1750
-Connection ~ 10050 1750
+	11900 1650 12250 1650
+Wire Wire Line
+	12250 1750 11900 1750
+Wire Wire Line
+	12250 1850 11900 1850
 Wire Wire Line
 	4050 1800 4250 1800
@@
 Wire Wire Line
 	4250 1900 4700 1900
+Wire Wire Line
+	8300 4100 8550 4100
+Wire Wire Line
+	8200 3750 8200 6600
+Wire Wire Line
+	8200 6600 10950 6600
+Wire Wire Line
+	10850 6700 8100 6700
+Wire Wire Line
+	8100 6700 8100 3750
+Wire Wire Line
+	7900 4100 7900 3750
+Wire Wire Line
+	8000 3750 8000 6500
+Wire Wire Line
+	8000 6500 11050 6500
+Wire Wire Line
+	9950 1150 8500 1150
 $EndSCHEMATC

Commit message: Add new version 2-way active filter.
Parts:
- added C45, C46, C47, C48: 0.047 мк, symbol CAPITORS
- C32, C33: value 2.2 мк -> 0.047 мк
Connections:
- net GND: now also XP3.1, C46.2, C47.2, C48.2; no longer C10.1, C9.2, DA1.2 (com), DA2.1 (com), TV1.11, TV1.8, XP3.6
- net AGND: now reaches C16.2, C17.1, C18.2, C19.1, XS2.2
- net AGND: now also C10.1, C9.2, DA1.2 (com), DA2.1 (com), TV1.11, TV1.8
- net at C24.2, R27.2, R27.3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: now also DA5.7 (OUT2); no longer DA5.1 (OUT1)
- net at C27.1, R61.1: now also DA5.11 (V-); no longer DA5.11 (V-)
- net at C25.2, R26.2, XP6.1: now also DA5.6 (~IN2); no longer DA5.2 (~IN1)
- net at R23.2, R25.1: now also DA5.5 (IN2); no longer DA5.3 (IN1)
- net at C26.1, R62.1: now also DA5.4 (V+); no longer DA5.4 (V+)
- net CAP3: now reaches C29.1, DA5.12 (IN4), R32.2, XP7.3
- net CAP3: now also C46.1, C47.1, C48.1
- net CAP1: now reaches C28.1, R29.2, R29.3, R30.1, XP7.2
- net CAP1: now also C32.1, C33.1, C45.1
- net CAP2: now reaches C28.2, DA5.13 (~IN4), DA5.14 (OUT4), R35.2
- net CAP2: now also C32.2, C33.2, R37.3, C45.2; no longer C33.1
- net at C30.2, R31.2, R33.1: now also DA5.3 (IN1); no longer DA5.5 (IN2)
- net at C31.1, R34.1, R35.1: now also DA5.2 (~IN1); no longer DA5.6 (~IN2)
- net at C31.2, R34.2: now also DA5.1 (OUT1), R36.3; no longer C32.1, DA5.7 (OUT2)
- net at DA3.1 (OUT1), DA3.2 (~IN1), R42.2: now also XP3.6; no longer XP3.1
- net at C20.2, DA6.14 (OUT4), R14.2: now also XP3.4; no longer XP3.3
- net at DA4.3 (IN1): now also XP3.2; no longer XP3.5
- net at R50.3: now also XP3.5; no longer XP3.2
- net at R49.3: now also XP3.3; no longer XP3.4
- net at XP11.1: now also R44.1; no longer R43.1
- net at XP11.4: now also R43.1; no longer R44.1
Other:
- moved on the sheet: C26, C27, C34, C35, R36, R37, R38, R39, R40, R41, R61, R62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

Commit message: Send to production of 2-way active filter.
Parts:
- renumbered XS9 to XP9
Changed lines of the file:
@@
 Sheet 1 1
 Title ""
-Date "12 sep 2015"
+Date "13 sep 2015"
 Rev ""
 Comp ""
@@
 P 21200 5400
 AR Path="/530320C3" Ref="XS?"  Part="1"
-AR Path="/557DF38E" Ref="XS9"  Part="1"
-F 0 "XS9" H 21250 5600 50  0000 L BNN
+AR Path="/557DF38E" Ref="XP9"  Part="1"
+F 0 "XP9" H 21250 5600 50  0000 L BNN
 F 1 "WF-4" H 21250 5500 50  0000 L BNN
 F 2 "~" H 21650 5550 50  0001 C CNN

Commit message: Moved to kicad 4.0.0
Parts:
- C1, C2, C3: footprint (none) -> LFcomponents:CAPACITOR_MKP4_27_5_32x11
- C10, C9: footprint (none) -> LFcomponents:CAPACITOR_10_D22
- C11, C12, C13, C14, C15, C18, C19, C20, C21, C26, C27, C30, C31, C34, C35, C36, C37, C38, C39, C4, C40, C41, C42, C43, C44, C5, C6, C7, C8, R1, R10, R11, R12, R13, R14, R15, R16, R17, R2, R21, R22, R23, R25, R26, R28, R3, R31, R32, R33, R34, R35, R38, R39, R4, R40, R41, R42, R43, R44, R45, R46, R47, R48, R5, R51, R52, R53, R54, R55, R56, R57, R58, R59, R6, R60, R61, R62, R63, R64, R7, R8, R9: footprint (none) -> LFsmd_case:SMD0805
- C16, C17: footprint (none) -> LFcomponents:CAPACITOR_CD263_2.54_D6.3
- C22, C23, C24, C25, C28, C29, C32, C33, C45, C46, C47, C48: footprint (none) -> LFcomponents:CAPACITOR_FKP2_5_7x6.5
- DA1, DA2: footprint (none) -> LFcomponents:TO220_RAD_16.5x15
- DA3, DA4, DA7: footprint ~ -> SOIC8~
- DA5, DA6: footprint ~ -> SOIC14~
- FU1: footprint ~ -> FU_PTF15B~
- R18, R19, R20, R24, R27, R29, R30, R36, R37, R49, R50: footprint (none) -> LFcomponents:Electron_3296W
- TV1: footprint (none) -> LFtransformator:BVEI_481_1120
- VD1, VD2, VD3, VD4: footprint (none) -> LFcomponents:DO-41
- XP1, XP2: footprint ~ -> WF-3~
- XP10, XP11, XP8, XP9: footprint ~ -> WF-4~
- XP3: footprint ~ -> WF-6~
- XP4, XP7: footprint ~ -> PIN_ARRAY_3x1~
- XP5, XP6: footprint ~ -> PIN_ARRAY_2x1~
- XS1: footprint ~ -> DG126-5.0-02P-14~
- XS2, XS3: footprint ~ -> DG126-5.0-03P-14~
