File: kicad/PS15100/PS15100.sch (KiCad schematic (older format))
At the start: 18 parts

Commit message: Развёл плату стабилизатора на +/-100В 15А.
Parts:
- C1, C2, C4, C5: footprint LFcomponents:CAPACITOR_10_D36 -> IWcomponents:CAPACITOR_10_D36
- C3, C6: footprint LFcomponents:K73-17 -> IWcomponents:K73-17
- FU1, FU2: footprint LFcomponents:FU_PTF15B -> IWcomponents:FU_PTF15B
- R1, R2: footprint LFcomponents:RESISTOR_1W -> IWcomponents:RESISTOR_1W
- VD1, VD2, VD3, VD4: footprint LFcomponents:TO220_RAD_16.5x15_VD -> IWcomponents:TO220_RAD_16.5x15_VD
- XS1: footprint LFcomponents:TO220_RAD_16.5x15_VD -> IWconnectors:DG126-5.0-03P-14
- XS2, XS3, XS4: footprint DG126-5.0-03P-14~ -> IWconnectors:DG126-5.0-03P-14
Changed lines of the file:
@@
 F 0 "C5" V 7475 4375 71  0000 C CNN
 F 1 "10000 мк 100 В" V 7575 4575 71  0000 C CNN
-F 2 "LFcomponents:CAPACITOR_10_D36" H 6850 4375 60  0001 C CNN
+F 2 "IWcomponents:CAPACITOR_10_D36" H 6850 4375 60  0001 C CNN
 F 3 "" H 6850 4375 60  0001 C CNN
 	1    6850 4375
@@
 F 0 "C2" V 6400 3550 71  0000 C CNN
 F 1 "10000 мк 100 В" V 6500 3775 71  0000 C CNN
-F 2 "LFcomponents:CAPACITOR_10_D36" H 6850 3550 60  0001 C CNN
+F 2 "IWcomponents:CAPACITOR_10_D36" H 6850 3550 60  0001 C CNN
 F 3 "" H 6850 3550 60  0001 C CNN
 	1    6850 3550
@@
 F 0 "C6" H 7600 4450 71  0000 C CNN
 F 1 "0.47мк 400В" H 7600 4350 71  0000 C CNN
-F 2 "LFcomponents:K73-17" H 7475 4625 60  0001 C CNN
+F 2 "IWcomponents:K73-17" H 7475 4625 60  0001 C CNN
 F 3 "" H 7475 4625 60  0001 C CNN
 	1    7475 4625
@@
 F 0 "C4" V 6650 4350 71  0000 C CNN
 F 1 "10000 мк 100 В" V 6750 4350 71  0000 C CNN
-F 2 "LFcomponents:CAPACITOR_10_D36" H 6025 4375 60  0001 C CNN
+F 2 "IWcomponents:CAPACITOR_10_D36" H 6025 4375 60  0001 C CNN
 F 3 "" H 6025 4375 60  0001 C CNN
 	1    6025 4375
@@
 F 0 "C1" V 5600 3550 71  0000 C CNN
 F 1 "10000 мк 100 В" V 5700 3525 71  0000 C CNN
-F 2 "LFcomponents:CAPACITOR_10_D36" H 6025 3525 60  0001 C CNN
+F 2 "IWcomponents:CAPACITOR_10_D36" H 6025 3525 60  0001 C CNN
 F 3 "" H 6025 3525 60  0001 C CNN
 	1    6025 3525
@@
 F 0 "C3" H 7600 3625 71  0000 C CNN
 F 1 "0.47мк 400В" H 7550 3500 71  0000 C CNN
-F 2 "LFcomponents:K73-17" H 7475 3775 60  0001 C CNN
+F 2 "IWcomponents:K73-17" H 7475 3775 60  0001 C CNN
 F 3 "" H 7475 3775 60  0001 C CNN
 	1    7475 3775
@@
 F 0 "XS3" H 8700 3750 50  0000 L BNN
 F 1 "DG126-5.0-03P-14" H 8400 3850 50  0000 L BNN
-F 2 "DG126-5.0-03P-14~" H 8900 4350 50  0001 C CNN
+F 2 "IWconnectors:DG126-5.0-03P-14" H 8900 4350 50  0001 C CNN
 F 3 "" H 8450 4200 60  0001 C CNN
 	1    8450 4200
@@
 F 0 "FU2" H 3850 4650 60  0000 C CNN
 F 1 "15 A" H 4150 4650 60  0000 C CNN
-F 2 "LFcomponents:FU_PTF15B" H 3900 4500 60  0001 C CNN
+F 2 "IWcomponents:FU_PTF15B" H 3900 4500 60  0001 C CNN
 F 3 "" H 3900 4500 60  0001 C CNN
 	1    3900 4500
@@
 F 0 "FU1" H 3850 3850 60  0000 C CNN
 F 1 "15 A" H 4150 3850 60  0000 C CNN
-F 2 "LFcomponents:FU_PTF15B" H 3900 3700 60  0001 C CNN
+F 2 "IWcomponents:FU_PTF15B" H 3900 3700 60  0001 C CNN
 F 3 "" H 3900 3700 60  0001 C CNN
 	1    3900 3700
@@
 F 0 "XS1" H 3600 4200 50  0000 L BNN
 F 1 "DG126-5.0-03P-14" H 3250 4100 50  0000 L BNN
-F 2 "LFcomponents:TO220_RAD_16.5x15_VD" H 3900 4150 50  0001 C CNN
+F 2 "IWconnectors:DG126-5.0-03P-14" H 3900 4150 50  0001 C CNN
 F 3 "" H 3450 4000 60  0001 C CNN
 	1    3450 4000
@@
 F 0 "XS2" H 8700 3050 50  0000 L BNN
 F 1 "DG126-5.0-03P-14" H 8400 3150 50  0000 L BNN
-F 2 "DG126-5.0-03P-14~" H 8900 3650 50  0001 C CNN
+F 2 "IWconnectors:DG126-5.0-03P-14" H 8900 3650 50  0001 C CNN
 F 3 "" H 8450 3500 60  0001 C CNN
 	1    8450 3500
@@
 F 0 "XS4" H 8700 4450 50  0000 L BNN
 F 1 "DG126-5.0-03P-14" H 8400 4550 50  0000 L BNN
-F 2 "DG126-5.0-03P-14~" H 8900 5050 50  0001 C CNN
+F 2 "IWconnectors:DG126-5.0-03P-14" H 8900 5050 50  0001 C CNN
 F 3 "" H 8450 4900 60  0001 C CNN
 	1    8450 4900
@@
 F 0 "R1" H 8350 3700 71  0000 C CNN
 F 1 "20 к" H 8050 3700 71  0000 C CNN
-F 2 "LFcomponents:RESISTOR_1W" H 8050 3550 60  0001 C CNN
+F 2 "IWcomponents:RESISTOR_1W" H 8050 3550 60  0001 C CNN
 F 3 "" H 8050 3550 60  0000 C CNN
 	1    8050 3550
@@
 F 0 "R2" H 8350 4550 71  0000 C CNN
 F 1 "20 к" H 8050 4550 71  0000 C CNN
-F 2 "LFcomponents:RESISTOR_1W" H 8050 4400 60  0001 C CNN
+F 2 "IWcomponents:RESISTOR_1W" H 8050 4400 60  0001 C CNN
 F 3 "" H 8050 4400 60  0000 C CNN
 	1    8050 4400
@@
 F 0 "VD1" H 4930 4130 71  0000 C CNN
 F 1 "MBR15100" H 4900 4000 71  0000 C CNN
-F 2 "LFcomponents:TO220_RAD_16.5x15_VD" H 4750 3850 60  0001 C CNN
+F 2 "IWcomponents:TO220_RAD_16.5x15_VD" H 4750 3850 60  0001 C CNN
 F 3 "" H 4750 3850 60  0000 C CNN
 	1    4750 3850
@@
 F 0 "VD2" H 5630 4130 71  0000 C CNN
 F 1 "MBR15100" H 5600 4000 71  0000 C CNN
-F 2 "LFcomponents:TO220_RAD_16.5x15_VD" H 5450 3850 60  0001 C CNN
+F 2 "IWcomponents:TO220_RAD_16.5x15_VD" H 5450 3850 60  0001 C CNN
 F 3 "" H 5450 3850 60  0000 C CNN
 	1    5450 3850
@@
 F 0 "VD3" H 4930 4930 71  0000 C CNN
 F 1 "MBR15100" H 4900 4800 71  0000 C CNN
-F 2 "LFcomponents:TO220_RAD_16.5x15_VD" H 4750 4650 60  0001 C CNN
+F 2 "IWcomponents:TO220_RAD_16.5x15_VD" H 4750 4650 60  0001 C CNN
 F 3 "" H 4750 4650 60  0000 C CNN
 	1    4750 4650
@@
 F 0 "VD4" H 5630 4930 71  0000 C CNN
 F 1 "MBR15100" H 5600 4800 71  0000 C CNN
-F 2 "LFcomponents:TO220_RAD_16.5x15_VD" H 5450 4650 60  0001 C CNN
+F 2 "IWcomponents:TO220_RAD_16.5x15_VD" H 5450 4650 60  0001 C CNN
 F 3 "" H 5450 4650 60  0000 C CNN
 	1    5450 4650

Commit message: Подготовил плату PS10015 к отправке на изготовление.
Parts:
- VD1, VD2, VD3, VD4: symbol DIOD_SCHTOTTKY_DUAL -> DIOD_SCHTOTTKY_DUAL-RESCUE-PS15100
Changed lines of the file:
@@
 EESchema Schematic File Version 2
+LIBS:PS15100-rescue
 LIBS:LFbutton
 LIBS:LFcapitors
@@
 Connection ~ 8050 4900
 $Comp
-L DIOD_SCHTOTTKY_DUAL VD1
+L DIOD_SCHTOTTKY_DUAL-RESCUE-PS15100 VD1
 U 1 1 56B75911
 P 4750 3850
@@
 $EndComp
 $Comp
-L DIOD_SCHTOTTKY_DUAL VD2
+L DIOD_SCHTOTTKY_DUAL-RESCUE-PS15100 VD2
 U 1 1 56B75B22
 P 5450 3850
@@
 $EndComp
 $Comp
-L DIOD_SCHTOTTKY_DUAL VD3
+L DIOD_SCHTOTTKY_DUAL-RESCUE-PS15100 VD3
 U 1 1 56B75C46
 P 4750 4650
@@
 $EndComp
 $Comp
-L DIOD_SCHTOTTKY_DUAL VD4
+L DIOD_SCHTOTTKY_DUAL-RESCUE-PS15100 VD4
 U 1 1 56B75C4C
 P 5450 4650
