File: kicad/timer_ne555/timer_ne555.sch (KiCad schematic (older format))
At the start: 17 parts

Commit message: Добавил в схему с реле времени на NE555 логику при срабатывание при не нулевом сопротивление контактов датчика.
Parts:
- added C1: 0.1 мк, symbol CAPITORS
- added DD1: 74AC08, symbol 74AC08
- added R1: 1 к, symbol RESISTOR_0_125W
- added R2, R3: 22 к, symbol RESISTOR_0_125W
- C4: renamed from C3; value 0.01 мк -> 0.1 мк
- XP2: renamed from XP1; symbol PIN_M_2 -> PIN_M_3
- XP3: symbol PIN_M_3 -> PIN_M_2
- renumbered C1 to C2, C2 to C3, R7 to R10, R8 to R11, R1 to R4, R2 to R5, R3 to R6, R4 to R7, R5 to R8, R6 to R9, XP2 to XP1
Connections:
- net GND: now also XP2.3, C1.2, DD1.7 (V-); no longer XP2.2
- net VCC: now also C1.1, DD1.14 (V+), R2.2, R3.1
- net at DA1.2 (TRIG), R4.1: now also DD1.3; no longer XP1.1
- net at VD1.1, VT1.3: now also XP3.2; no longer XP3.3
- new net: R1.1, XP1.1
- new net: DD1.1, R1.2, R2.1
- new net: DD1.2, R3.2
Other:
- note added: "*DD1 служит для срабатывания реле времени если сопротивление\nконтактов перемыкаюших контакты разъёма XP1 достигает 3 кОм\n"
- note added: "*К кнопке запуска\n таймера"
- note added: "К источнику\nпостоянного\n тока 5 В"
- note removed: "К источнику питания\n от 5 В до 18 В"
- note removed: "К кнопке запуска\n таймера"
- moved on the sheet: C2, C3, C4, DA1, R10, R11, R4, R5, R6, R7, R8, R9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
