File: kicad/mark_III_amp/mark_III_amp.sch (KiCad schematic (older format))
At the start: 119 parts

Commit message: Добавил новую версию усилителя mc_amplifier_rev_1.
Parts:
- added C?: 22 мк 35 В, symbol CAPITORS_ELECTROLYTIC
Connections:
- net at C4.1, R6.2, VT1.1: now also C?.2
- net at C4.2, R8.2, R9.1: now also C?.1
Changed lines of the file:
@@
 	3700 3550 3950 3550
 Wire Wire Line
-	3850 3550 3850 3700
+	3850 3100 3850 3700
 Connection ~ 3850 3550
 Wire Wire Line
@@
 	3250 4150 3250 4400
 Wire Wire Line
-	3250 3950 3250 3550
+	3250 3100 3250 3950
 Connection ~ 3250 3550
 Wire Wire Line
@@
 Wire Wire Line
 	11150 4650 12350 4650
+$Comp
+L CAPITORS_ELECTROLYTIC C?
+U 1 1 5B4CE2EA
+P 3700 3100
+F 0 "C?" H 3800 3350 71  0000 C CNN
+F 1 "22 мк 35 В" H 3850 3250 71  0000 C CNN
+F 2 "" H 3700 3100 60  0000 C CNN
+F 3 "" H 3700 3100 60  0000 C CNN
+	1    3700 3100
+	-1   0    0    -1
+$EndComp
+Wire Wire Line
+	3250 3100 3450 3100
+Wire Wire Line
+	3700 3100 3850 3100
 $EndSCHEMATC
