File: kicad/active_low-pass_filter/active_low-pass_filter.sch (KiCad schematic (older format))
At the start: 70 parts

Commit message: Поправлил схему фильтров active_low-pass_filter.
Parts:
- removed R19: 10 к, symbol RESISTOR_TRIMMING
- removed R22, R8, R9: 50 к, symbol RESISTOR_TRIMMING
- removed R25: 250, symbol RESISTOR
- added C17: 1 мк, symbol LFcapitors:CAPITORS
- added C20: 0.47 мк, symbol LFcapitors:CAPITORS
- added R15, R17: 1 к, symbol LFresistor:RESISTOR
- added R16, R18, R19, R20: 50 к, symbol LFresistor:RESISTOR_TRIMMING
- added XP3: WF-4, ~, symbol LFconnectors:connector_5pin_gost
- added XP4, XP5, XP6, XP7: WF-2, ~, symbol LFconnectors:connector_2pin_gost
- added XP8, XP9: WF-3, ~, symbol LFconnectors:connector_3pin_gost
- C1: renamed from C9; symbol CAPITORS -> LFcapitors:CAPITORS
- C10: renamed from C25; symbol CAPITORS -> LFcapitors:CAPITORS
- C11: renamed from C2; symbol CAPITORS_ELECTROLYTIC -> LFcapitors:CAPITORS_ELECTROLYTIC
- C12: renamed from C5; symbol CAPITORS_ELECTROLYTIC -> LFcapitors:CAPITORS_ELECTROLYTIC
- C13: renamed from C21; symbol CAPITORS -> LFcapitors:CAPITORS
- C14: renamed from C23; symbol CAPITORS -> LFcapitors:CAPITORS
- C15: renamed from C3; symbol CAPITORS -> LFcapitors:CAPITORS
- C16: renamed from C6; symbol CAPITORS -> LFcapitors:CAPITORS
- C18: renamed from C14; symbol CAPITORS -> LFcapitors:CAPITORS
- C19: renamed from C17; symbol CAPITORS -> LFcapitors:CAPITORS
- C2: renamed from C19; symbol CAPITORS -> LFcapitors:CAPITORS
- C21: renamed from C8; symbol CAPITORS -> LFcapitors:CAPITORS
- C22: symbol CAPITORS -> LFcapitors:CAPITORS
- C23: renamed from C10; symbol CAPITORS -> LFcapitors:CAPITORS
- C24: renamed from C27; symbol CAPITORS -> LFcapitors:CAPITORS
- C25: renamed from C28; symbol CAPITORS -> LFcapitors:CAPITORS
- C26: renamed from C15; symbol CAPITORS -> LFcapitors:CAPITORS
- C27: renamed from C18; symbol CAPITORS -> LFcapitors:CAPITORS
- C28: renamed from C26; symbol CAPITORS -> LFcapitors:CAPITORS
- C29: renamed from C7; symbol CAPITORS -> LFcapitors:CAPITORS
- C3: renamed from C11; symbol CAPITORS -> LFcapitors:CAPITORS
- C30: renamed from C12; symbol CAPITORS -> LFcapitors:CAPITORS
- C4: renamed from C20; symbol CAPITORS -> LFcapitors:CAPITORS
- C5: renamed from C1; symbol CAPITORS_ELECTROLYTIC -> LFcapitors:CAPITORS_ELECTROLYTIC
- C6: renamed from C4; symbol CAPITORS_ELECTROLYTIC -> LFcapitors:CAPITORS_ELECTROLYTIC
- C7: renamed from C13; symbol CAPITORS -> LFcapitors:CAPITORS
- C8: renamed from C24; symbol CAPITORS -> LFcapitors:CAPITORS
- C9: renamed from C16; symbol CAPITORS -> LFcapitors:CAPITORS
- DA1: renamed from DA3; symbol LM258 -> LFcomponents:LM258
- DA2: renamed from DA6; symbol LM258 -> LFcomponents:LM258
- DA3: renamed from DA1; symbol 7815 -> LFcomponents:7815
- DA4: renamed from DA2; symbol 7915 -> LFcomponents:7915
- DA5: renamed from DA4; symbol LM258 -> LFcomponents:LM258
- DA6: renamed from DA7; symbol LM258 -> LFcomponents:LM258
- DA7: renamed from DA5; symbol LM258 -> LFcomponents:LM258
- R1: renamed from R12; symbol RESISTOR -> LFresistor:RESISTOR
- R10: renamed from R17; symbol RESISTOR -> LFresistor:RESISTOR
- R11: renamed from R21; symbol RESISTOR -> LFresistor:RESISTOR
- R12: renamed from R13; symbol RESISTOR -> LFresistor:RESISTOR
- R13: renamed from R2; symbol RESISTOR -> LFresistor:RESISTOR
- R14: renamed from R5; value 5.6 к -> 1 к; symbol RESISTOR -> LFresistor:RESISTOR
- R2: renamed from R15; symbol RESISTOR -> LFresistor:RESISTOR
- R21: renamed from R23; symbol RESISTOR -> LFresistor:RESISTOR
- R22: renamed from R6; value 5.6 к -> 1 к; symbol RESISTOR -> LFresistor:RESISTOR
- R23: renamed from R18; symbol RESISTOR -> LFresistor:RESISTOR
- R24: renamed from R7; symbol RESISTOR -> LFresistor:RESISTOR
- R25: renamed from R24; value 1 к -> 5.1 к; symbol RESISTOR -> LFresistor:RESISTOR
- R26: renamed from R10; symbol RESISTOR -> LFresistor:RESISTOR
- R3: value 10 к -> 220; symbol RESISTOR -> LFresistor:RESISTOR
- R4: renamed from R14; value 10 к -> 220; symbol RESISTOR -> LFresistor:RESISTOR
- R5: renamed from R16; symbol RESISTOR -> LFresistor:RESISTOR
- R6: renamed from R20; symbol RESISTOR -> LFresistor:RESISTOR
- R7: renamed from R4; symbol RESISTOR -> LFresistor:RESISTOR
- R8: renamed from R11; symbol RESISTOR -> LFresistor:RESISTOR
- R9: renamed from R1; symbol RESISTOR -> LFresistor:RESISTOR
- TV1: symbol BVEI_302_2028 -> LFtransformator:BVEI_302_2028
- VD1, VD4: symbol SHOTTKY_DIODE -> LFdiod:SHOTTKY_DIODE
- VD2: renamed from VD3; symbol SHOTTKY_DIODE -> LFdiod:SHOTTKY_DIODE
- VD3: renamed from VD2; symbol SHOTTKY_DIODE -> LFdiod:SHOTTKY_DIODE
- XP1: renamed from XS2; symbol PIN_F_4 -> LFconnectors:connector_4pin_gost
- XP2: renamed from XS3; symbol PIN_F_4 -> LFconnectors:connector_4pin_gost
- XS1: symbol PIN_F_2 -> LFconnectors:connector_2pin_gost
- XS2: renamed from XS4; value WF-2 -> WP-2; symbol PIN_F_2 -> LFconnectors:connector_2pin_gost
- XS3: renamed from XS5; symbol PIN_F_2 -> LFconnectors:connector_2pin_gost
Connections:
- net GND: now also R18.1, XP3.1, XP4.2, XP8.3
- net at R24.2: now also XP9.1
- net at C29.2: now also XP9.2
- net at R26.1: now also XP9.3
- net at DA6.1 (OUT1), R23.2: now also C17.1
- net at C22.2, DA6.3 (IN1): now also XP3.2
- net at DA6.5 (IN2): now also C20.2, R17.1
- net at DA6.6 (~IN2): now also DA6.7 (OUT2), R19.2, R19.3, XP5.1, XP8.1
- net at C28.1: now also XP8.2
- new net: R14.2, R16.1, XP6.1
- new net: R20.2, R20.3, R22.1, XP7.2
- new net: C21.1, R16.2, R16.3, R20.1, XP6.2, XP7.1
- new net: C17.2, C20.1, R15.1
- new net: R15.2, R19.1, XP5.2
- new net: R17.2, R18.2, R18.3, XP4.1
Other:
- note added: "220 В"
- note added: "GND"
- note added: "LED+"
- note added: "LED-"
- note added: "К РЕЗИСТОРУ 10 кОм"
- note added: "К РЕЗИСТОРУ 10 кОм\n(РЕГУЛИРОВКА ГРОМКОСТИ)"
- note added: "К СДВОЕННОМУ\nРЕЗИСТОРУ 50 кОм"
- note added: "К светодиоду"
- note added: "ЛК"
- note added: "ЛК+ПК"
- note added: "ПК"
- note added: "ПОВТОРИТЕЛИ"
- note added: "Ползунок"
- note added: "ФИЛЬТР ВЧ \n (настроен на 50 Гц -3Дб)"
- note added: "ФИЛЬТР НЧ \n (настраивется на 50-200 Гц -3Дб)"
- note added: "ФИЛЬТР НЧ \n (настроен на 300 Гц -3Дб)"
- note removed: "220 V"
- note removed: "К светодиоду\n(5 В, 15 мА)"
- note removed: "ПОВТОРИТЕЛЬ"
- note removed: "ФИЛЬТР НЧ \n (настроен на 400 Гц -3Дб)"
- note removed: "ФИЛЬТР НЧ \n (настроен на 50-200 Гц -3Дб)"
- moved on the sheet: C13, C14, C19, C23, C26, C27, C28, C29, C30, R10, R11, R14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

Commit message: Добавил конденсаторы в повторитель сабвуферного фильтра для удаления самопроизвольного возмбуждения каскада.
Parts:
- added C31, C32: 22 п, symbol LFcapitors:CAPITORS
Connections:
- net GND: now also C31.2
- net at DA5.3 (IN1), R12.2, R7.2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: now also C31.1
- net at DA5.1 (OUT1), R13.2, R14.1: now also C32.2
- net at DA5.2 (~IN1), R13.1, R9.1: now also C32.1
Other:
- note added: "К СДВОЕННОМУ\nЛОГАРИФМИЧЕСКОМУ\n РЕЗИСТОРУ 50 кОм"
- note added: "НЕИНВЕРТИРУЮЩИЙ\n СУММАТОР"
- note removed: "К СДВОЕННОМУ\nРЕЗИСТОРУ 50 кОм"
- note removed: "СУММАТОР\nНЕИНВЕРТИРУЮЩИЙ"
- moved on the sheet: R12
Changed lines of the file:
@@
 	6000 3950 6350 3950
 Wire Wire Line
-	6900 4950 6900 4700
+	6900 4900 6900 4800
 Wire Wire Line
 	6900 4700 6900 4400
@@
 Connection ~ 7100 3950
 Wire Wire Line
-	6900 5200 6900 5450
+	6900 5150 6900 5250
 Wire Wire Line
 	8700 4400 8800 4400
@@
 Wire Wire Line
 	7100 3950 6600 3950
-Wire Wire Line
-	6600 4700 6900 4700
 Connection ~ 6900 4700
 Connection ~ 6900 4400
@@
 	1    0    0    -1
 $EndComp
-Text Label 6900 5450 1    60   ~ 0
+Text Label 6900 5500 1    60   ~ 0
 GND
 $Comp
 L LFresistor:RESISTOR R12
 U 1 1 530DA6ED
-P 6900 5200
-F 0 "R12" V 7100 5450 71  0000 C CNN
-F 1 "100 к" V 6950 5450 71  0000 C CNN
-F 2 "" H 6900 5200 60  0001 C CNN
-F 3 "" H 6900 5200 60  0001 C CNN
-	1    6900 5200
+P 6900 5150
+F 0 "R12" V 7150 4950 71  0000 C CNN
+F 1 "100 к" V 6950 4900 71  0000 C CNN
+F 2 "" H 6900 5150 60  0001 C CNN
+F 3 "" H 6900 5150 60  0001 C CNN
+	1    6900 5150
 	0    -1   -1   0
 $EndComp
@@
           ФИЛЬТР НЧ \n (настроен на 300 Гц -3Дб)
 Text Notes 6950 3300 0    120  ~ 0
-     СУММАТОР\nНЕИНВЕРТИРУЮЩИЙ
+НЕИНВЕРТИРУЮЩИЙ\n     СУММАТОР
 $Comp
 L LFcomponents:LM258 DA7
@@
 U 1 1 604D5D90
 P 9900 4400
-F 0 "R20" H 9850 4600 71  0000 C CNN
+F 0 "R20" H 9900 4600 71  0000 C CNN
 F 1 "50 к" H 10200 4600 71  0000 C CNN
 F 2 "" H 9900 4400 60  0001 C CNN
@@
 Wire Wire Line
 	14350 4400 14650 4400
-Text Notes 13800 5950 0    60   ~ 0
-  К СДВОЕННОМУ\nРЕЗИСТОРУ 50 кОм
+Text Notes 13800 6050 0    60   ~ 0
+   К СДВОЕННОМУ\nЛОГАРИФМИЧЕСКОМУ\n РЕЗИСТОРУ 50 кОм
 $Comp
 L LFconnectors:connector_5pin_gost XP3
@@
 Text Notes 6650 10850 0    120  ~ 0
           ФИЛЬТР   ВЧ \n (настроен на 50 Гц -3Дб)
+$Comp
+L LFcapitors:CAPITORS C32
+U 1 1 603B55F3
+P 7800 3650
+F 0 "C32" H 7950 3950 71  0000 C CNN
+F 1 "22 п" H 7950 3800 71  0000 C CNN
+F 2 "" H 7800 3650 60  0001 C CNN
+F 3 "" H 7800 3650 60  0001 C CNN
+	1    7800 3650
+	1    0    0    -1
+$EndComp
+Wire Wire Line
+	8050 3650 8800 3650
+Wire Wire Line
+	8800 3650 8800 3950
+Connection ~ 8800 3950
+Wire Wire Line
+	7800 3650 7100 3650
+Wire Wire Line
+	7100 3650 7100 3950
+$Comp
+L LFcapitors:CAPITORS C31
+U 1 1 604149E5
+P 6700 4900
+F 0 "C31" V 6750 4600 71  0000 C CNN
+F 1 "22 п" V 6900 4650 71  0000 C CNN
+F 2 "" H 6700 4900 60  0001 C CNN
+F 3 "" H 6700 4900 60  0001 C CNN
+	1    6700 4900
+	0    1    1    0
+$EndComp
+Wire Wire Line
+	6600 4700 6900 4700
+Wire Wire Line
+	6700 4900 6700 4800
+Wire Wire Line
+	6700 4800 6900 4800
+Connection ~ 6900 4800
+Wire Wire Line
+	6900 4800 6900 4700
+Wire Wire Line
+	6700 5150 6700 5250
+Wire Wire Line
+	6700 5250 6900 5250
+Connection ~ 6900 5250
+Wire Wire Line
+	6900 5250 6900 5500
 $EndSCHEMATC
