File: kicad/mc_power_supply/mc_power_supply.kicad_pcb (KiCad board)
At the start: 2 copper layers, 118 x 65 mm, 26 parts

Commit message: Повторно отправил плату mm_power_supply_v3 в производство.
Changed lines of the file:
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@@
   )
   (setup
-    (last_trace_width 1)
+    (last_trace_width 0.25)
     (user_trace_width 0.5)
     (user_trace_width 1)
@@
     (visible_elements FFFFFF7F)
     (pcbplotparams
-      (layerselection 0x010e0_ffffffff)
+      (layerselection 0x00020_7ffffffe)
       (usegerberextensions false)
-      (usegerberattributes true)
-      (usegerberadvancedattributes true)
-      (creategerberjobfile true)
+      (usegerberattributes false)
+      (usegerberadvancedattributes false)
+      (creategerberjobfile false)
       (excludeedgelayer true)
       (linewidth 0.100000)
@@
     (add_net "Net-(TV1-Pad9)")
   )
+  (module IWsmd_case:SMD2512 (layer F.Cu)
+    (at 117.094 90.932 270)
+    (tags "CMS SM")
+    (attr smd)
+    (fp_text reference R1 (at -5.588 0) (layer F.SilkS)
+      (effects (font (size 0.762 0.762) (thickness 0.127)))
+    )
+    (fp_text value "510 к" (at 0.254 3.048 90) (layer F.SilkS) hide
+      (effects (font (size 1.016 0.762) (thickness 0.127)))
+    )
+    (fp_line (start 4.572 -2.286) (end 4.572 2.286) (layer F.SilkS) (width 0.127))
+    (fp_line (start -4.572 2.286) (end -4.572 -2.286) (layer F.SilkS) (width 0.127))
+    (fp_line (start -4.572 -2.286) (end 4.572 -2.286) (layer F.SilkS) (width 0.127))
+    (fp_line (start -4.572 2.286) (end 4.572 2.286) (layer F.SilkS) (width 0.127))
+    (pad 2 smd rect (at 3.25 0 270) (size 1.9 3.8) (layers F.Cu F.Paste F.Mask)
+      (net 2 "Net-(C1-Pad1)"))
+    (pad 1 smd rect (at -3.25 0 270) (size 1.9 3.8) (layers F.Cu F.Paste F.Mask)
+      (net 1 "Net-(C1-Pad2)"))
+    (model smd/chip_cms.wrl
+      (at (xyz 0 0 0))
+      (scale (xyz 0.21 0.3 0.2))
+      (rotate (xyz 0 0 0))
+    )
+  )
   (module IWsmd_case:TO-263-3_TabPin_2 (layer F.Cu)
     (at 193.802 114.681)
@@
       (rotate (xyz 0 0 0))
     )
-  )
-  (module IWsmd_case:SMD2512 (layer F.Cu)
-    (at 117.094 90.932 270)
-    (tags "CMS SM")
-    (attr smd)
-    (fp_text reference R1 (at -5.588 0) (layer F.SilkS)
-      (effects (font (size 0.762 0.762) (thickness 0.127)))
-    )
-    (fp_text value "510 к" (at 0.254 3.048 90) (layer F.SilkS) hide
-      (effects (font (size 1.016 0.762) (thickness 0.127)))
-    )
-    (fp_line (start -4.318 2.032) (end 4.318 2.032) (layer F.SilkS) (width 0.127))
-    (fp_line (start -4.318 -2.032) (end 4.318 -2.032) (layer F.SilkS) (width 0.127))
-    (fp_line (start -4.318 2.032) (end -4.318 -2.032) (layer F.SilkS) (width 0.127))
-    (fp_line (start 4.318 -2.032) (end 4.318 2.032) (layer F.SilkS) (width 0.127))
-    (pad 2 smd rect (at 3.25 0 270) (size 1.9 3.8) (layers F.Cu F.Paste F.Mask)
-      (net 2 "Net-(C1-Pad1)"))
-    (pad 1 smd rect (at -3.25 0 270) (size 1.9 3.8) (layers F.Cu F.Paste F.Mask)
-      (net 1 "Net-(C1-Pad2)"))
-    (model smd/chip_cms.wrl
-      (at (xyz 0 0 0))
-      (scale (xyz 0.21 0.3 0.2))
-      (rotate (xyz 0 0 0))
-    )

Commit message: Успешно изготовил и проверил первый экземляр платы MM_power_supply_ver. 3.0
Parts:
- DA1: value LM317D2T-TR -> LM317KTTR
