File: kicad/adjustable_mm_amplifier/adjustable_mm_amplifier.sch (KiCad schematic (older format))
At the start: 23 parts

Commit message: Закончил разрабатывать схему усилителя для микрофонов.
Parts:
- removed C?: 47 мк 63 В, symbol LFcapitors:CAPITORS_ELECTROLYTIC
- removed C?: 22 п, symbol LFcapitors:CAPITORS
- removed R? (x3): 1 к 1%, symbol LFresistor:RESISTOR
- removed R?: 50 к, symbol LFresistor:RESISTOR_TRIMMING
- added C7: 47 мк 63 В, symbol LFcapitors:CAPITORS_ELECTROLYTIC
- added C8: 22 п, symbol LFcapitors:CAPITORS
- added R10, R11, R12, R4: 1 к 1%, symbol LFresistor:RESISTOR
- added R13, R14, R7: 50 к, symbol LFresistor:RESISTOR_TRIMMING
- added R3, R9: 100 к, symbol LFresistor:RESISTOR
- added SB1, SB2, SB3, SB4: MTS-102-C4-R, symbol LFbutton:MTS-102-C4-R
- C6: renamed from C?; value 10 мк 25 В -> 10 мк 63 В
- DA1: value NE5532AD -> ADA4522-1ARZ
- gave numbers to parts that had none: 14
- renumbered XS to XS1
Connections:
- net GND: now also C7.2, R3.2, R9.2
- net at C4.1, DA1.1 (OUT1), R6.2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: now also R7.2, R7.3, SB1.1, SB3.2; no longer DA1.5 (IN2)
- net at C4.2, DA1.2 (~IN1), R5.1: now also R4.1
- net at C2.1, R2.2: now also SB1.2; no longer DA1.3 (IN1)
- net at DA1.6 (~IN2): now also C8.2, R10.1, R11.1, R12.1
- net at C9.1, DA1.7 (OUT2): now also C8.1, R13.2, R13.3, R14.2, R14.3, SB3.1
- net at R5.2, R6.1: now also SB2.3
- net at C3.1: now also R4.2
- new net: DA1.3 (IN1), R3.1, SB1.3
- new net: DA1.5 (IN2), R9.1, SB3.3
- new net: R7.1, SB2.2
- new net: R12.2, R13.1, SB4.3
- new net: C7.1, R10.2, R11.2
- new net: R14.1, SB4.2
Other:
- moved on the sheet: C1, C2, C3, C4, C5, C6, C9, DA1A, DA1B, R1, R15, R16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

Commit message: Продолжил разрабатывать плату микрофонного услителя на +9...+48.
Parts:
- removed R10: 1 к 1%, symbol LFresistor:RESISTOR
- removed R14: 50 к, symbol LFresistor:RESISTOR_TRIMMING
- removed SB4: MTS-102-C4-R, symbol LFbutton:MTS-102-C4-R
- C1: value 47 мк 63В -> 47 мк 63 В
- C2, C4, C5, C8, R1, R2, R3, R4, R5, R8, R9: footprint (none) -> IWsmd_case:SMD0805
- DA1: footprint (none) -> IWsmd_case:SOIC8
- R10: renamed from R11; footprint (none) -> IWsmd_case:SMD0805
- R11: renamed from R12; footprint (none) -> IWsmd_case:SMD0805
- R12: renamed from R13; footprint (none) -> IWsmd_case:BOURNS_3224J
- R13: renamed from R15; footprint (none) -> IWsmd_case:SMD0805
- R14: renamed from R16; footprint (none) -> IWsmd_case:SMD0805
- R6, R7: footprint (none) -> IWsmd_case:BOURNS_3224J
- XP1: value Neutrik XLR-M -> Neutrik NC3MAAH
- XS1: value Neutrik XLR-F -> Neutrik NC3FAH1
Other:
- note added: "+48 В"
- note added: "GND"
- note added: "ВХОД"
- note added: "ВЫХОД"
- note added: "Усилитель на 10, 20 дБ"
- note added: "Усилитель на 20 дБ"
- moved on the sheet: C3, C7, R10, R11, R12, R4

Commit message: Продолжил разрабатывать плату микрофонного услителя на +9...+48.
Parts:
- C9: value 47 мк 63В -> 47 мк 63 В
Changed lines of the file:
@@
 P 8550 2400
 F 0 "C9" H 8600 2700 71  0000 C CNN
-F 1 "47 мк 63В" H 8650 2600 71  0000 C CNN
+F 1 "47 мк 63 В" H 8650 2600 71  0000 C CNN
 F 2 "" H 8550 2400 50  0001 C CNN
 F 3 "" H 8550 2400 50  0001 C CNN

Commit message: Продолжил разрабатывать adjustable_mm_amplifier.
Parts:
- removed R7: 50 к, IWsmd_case:BOURNS_3224J, symbol LFresistor:RESISTOR_TRIMMING
- removed SB2: MTS-102-C4-R, symbol LFbutton:MTS-102-C4-R
- R1: value 47 к -> 100 к
- XP1: footprint (none) -> audio:Jack_XLR_Neutrik_NC3MAAH_Horizontal
- XS1: footprint (none) -> audio:Jack_XLR_Neutrik_NC4FAH_Horizontal; symbol LFconnectors:connector_4pin_gost -> LFconnectors:connector_3pin_gost
- renumbered R11 to R10, R12 to R11, R13 to R12, R14 to R13, R8 to R7, R9 to R8, R10 to R9, SB3 to SB2
Connections:
- net GND: no longer XS1.4
Other:
- note added: "Усиление 10 дБ"
- note added: "Усиление 20 дБ"
- note removed: "Усилитель на 10, 20 дБ"
- note removed: "Усилитель на 20 дБ"
- moved on the sheet: C3, C7, R4, R5, R6, R9
Changed lines of the file:
@@
 $EndDescr
 $Comp
-L LFconnectors:connector_4pin_gost XS1
+L LFconnectors:connector_3pin_gost XS1
 U 1 1 602FB9CD
 P 1650 2200
 F 0 "XS1" H 2017 2563 71  0000 C CNN
 F 1 "Neutrik NC3FAH1" H 2017 2440 71  0000 C CNN
-F 2 "" H 2000 2350 50  0001 C CNN
+F 2 "audio:Jack_XLR_Neutrik_NC4FAH_Horizontal" H 2000 2350 50  0001 C CNN
 F 3 "" H 1650 2200 60  0000 C CNN
 	1    1650 2200
@@
 F 0 "XP1" H 10090 2750 71  0000 L CNN
 F 1 "Neutrik NC3MAAH" H 9740 2620 71  0000 L CNN
-F 2 "" H 10150 2450 50  0001 C CNN
+F 2 "audio:Jack_XLR_Neutrik_NC3MAAH_Horizontal" H 10150 2450 50  0001 C CNN
 F 3 "" H 9800 2300 60  0000 C CNN
 	1    9800 2300
@@
 $EndComp
 $Comp
-L LFresistor:RESISTOR R8
+L LFresistor:RESISTOR R7
 U 1 1 60309AA4
 P 5500 2900
-F 0 "R8" H 5500 3000 71  0000 C CNN
+F 0 "R7" H 5500 3000 71  0000 C CNN
 F 1 "4.7" H 5750 3000 71  0000 C CNN
 F 2 "IWsmd_case:SMD0805" H 5500 2900 60  0001 C CNN
@@
 P 2550 2400
 F 0 "R1" V 2650 2700 71  0000 R CNN
-F 1 "47 к" V 2750 2750 71  0000 R CNN
+F 1 "100 к" V 2750 2800 71  0000 R CNN
 F 2 "IWsmd_case:SMD0805" H 2550 2400 60  0001 C CNN
 F 3 "AmpliOp.sch" V 2798 2322 60  0001 R CNN
@@
 Text Label 2000 2200 2    50   ~ 0
 GND
-Wire Wire Line
-	1650 2200 1750 2200
 Text Label 5600 2700 2    50   ~ 0
 GND
@@
 Text Label 2000 2400 2    50   ~ 0
 +Vcc
-Wire Wire Line
-	1650 2500 1750 2500
-Wire Wire Line
-	1750 2500 1750 2200
-Connection ~ 1750 2200
-Wire Wire Line
-	1750 2200 2000 2200
 $Comp
 L LFresistor:RESISTOR R5
 U 1 1 60364267
-P 3850 3800
-F 0 "R5" H 3950 4050 71  0000 C CNN
-F 1 "1 к 1%" H 4000 3950 71  0000 C CNN
-F 2 "IWsmd_case:SMD0805" H 3850 3800 60  0001 C CNN
-F 3 "AmpliOp.sch" H 3975 3931 60  0001 C CNN
-	1    3850 3800
+P 4000 3800
+F 0 "R5" H 4100 4050 71  0000 C CNN
+F 1 "1 к 1%" H 4150 3950 71  0000 C CNN
+F 2 "IWsmd_case:SMD0805" H 4000 3800 60  0001 C CNN
+F 3 "AmpliOp.sch" H 4125 3931 60  0001 C CNN
+	1    4000 3800
 	1    0    0    -1
 $EndComp
@@
 L LFcapitors:CAPITORS_ELECTROLYTIC C3
 U 1 1 6036975D
-P 3700 4600
-F 0 "C3" V 3750 4450 71  0000 R CNN
-F 1 "47 мк 63 В" V 3850 4500 71  0000 R CNN
-F 2 "" H 3700 4600 50  0001 C CNN
-F 3 "" H 3700 4600 50  0001 C CNN
-	1    3700 4600
-	0    -1   1    0
-$EndComp
-Wire Wire Line
-	3700 4850 3700 5050
-Text Label 3700 5050 1    50   ~ 0
+P 3700 4450
+F 0 "C3" V 3750 4300 71  0000 R CNN
+F 1 "47 мк 63 В" V 3850 4350 71  0000 R CNN
+F 2 "" H 3700 4450 50  0001 C CNN
+F 3 "" H 3700 4450 50  0001 C CNN
+	1    3700 4450
+	0    -1   1    0
+$EndComp
+Wire Wire Line
+	3700 4700 3700 4900
+Text Label 3700 4900 1    50   ~ 0
 GND
 Wire Wire Line
@@
 Wire Wire Line
 	5350 2400 5350 3400
-$Comp
-L LFresistor:RESISTOR_TRIMMING R6
-U 1 1 60388BE5
-P 4800 3800
-F 0 "R6" H 4900 4100 71  0000 C CNN
-F 1 "50 к" H 4900 4000 71  0000 C CNN
-F 2 "IWsmd_case:BOURNS_3224J" H 4800 3800 60  0001 C CNN
-F 3 "AmpliOp.sch" H 4925 4031 60  0001 C CNN
-	1    4800 3800
-	1    0    0    -1
-$EndComp
-Wire Wire Line
-	5050 3800 5200 3800
-Connection ~ 5350 3800
-Wire Wire Line
-	5050 3700 5200 3700
-Wire Wire Line
-	5200 3700 5200 3800
-Connection ~ 5200 3800
-Wire Wire Line
-	5200 3800 5350 3800
 Wire Wire Line
 	6650 2600 6750 2600
@@
 $EndComp
 $Comp
-L LFresistor:RESISTOR R14
+L LFresistor:RESISTOR R13
 U 1 1 603CDEB7
 P 9350 2500
-F 0 "R14" V 9450 2800 71  0000 R CNN
+F 0 "R13" V 9450 2800 71  0000 R CNN
 F 1 "10 к 1%" V 9550 3050 71  0000 R CNN
 F 2 "IWsmd_case:SMD0805" H 9350 2500 60  0001 C CNN
@@
 $EndComp
 $Comp
-L LFresistor:RESISTOR R13
+L LFresistor:RESISTOR R12
 U 1 1 603CDEC1
 P 8950 2400
-F 0 "R13" H 9100 2650 71  0000 C CNN
+F 0 "R12" H 9100 2650 71  0000 C CNN
 F 1 "100" H 9100 2550 71  0000 C CNN
 F 2 "IWsmd_case:SMD0805" H 8950 2400 60  0001 C CNN
@@
 Wire Wire Line
 	3700 3400 3700 3800
-$Comp
-L LFresistor:RESISTOR_TRIMMING R7
-U 1 1 6032DAA3
-P 4800 4250
-F 0 "R7" H 4900 4550 71  0000 C CNN
-F 1 "50 к" H 4900 4450 71  0000 C CNN
-F 2 "IWsmd_case:BOURNS_3224J" H 4800 4250 60  0001 C CNN
-F 3 "AmpliOp.sch" H 4925 4481 60  0001 C CNN
-	1    4800 4250
-	1    0    0    -1
-$EndComp
-Wire Wire Line
-	5050 4250 5200 4250
-Wire Wire Line
-	5050 4150 5200 4150
-Wire Wire Line
-	5200 4150 5200 4250
-Connection ~ 5200 4250
-Wire Wire Line
-	5200 4250 5350 4250
-Wire Wire Line
-	5350 3800 5350 4250
-Wire Wire Line
-	3700 3800 3850 3800
-Wire Wire Line
-	4800 3800 4250 3800
-$Comp
-L LFbutton:MTS-102-C4-R SB2
-U 1 1 603483CF
-P 4500 4250
-F 0 "SB2" H 4500 4050 70  0000 C CNN
-F 1 "MTS-102-C4-R" H 4500 3950 70  0000 C CNN
-F 2 "" V 4450 4150 60  0001 C CNN
-F 3 "" V 4450 4150 60  0000 C CNN
-	1    4500 4250
-	1    0    0    -1
-$EndComp
-Wire Wire Line
-	4700 4250 4800 4250
-Connection ~ 4250 3800
-Wire Wire Line
-	4250 3800 4100 3800
+Wire Wire Line
+	3700 3800 4000 3800
 Wire Wire Line
 	8200 2400 8300 2400
@@
 L LFcapitors:CAPITORS_ELECTROLYTIC C7
 U 1 1 60358AE1
-P 6650 4600
-F 0 "C7" V 6700 4450 71  0000 R CNN
-F 1 "47 мк 63 В" V 6800 4500 71  0000 R CNN
-F 2 "" H 6650 4600 50  0001 C CNN
-F 3 "" H 6650 4600 50  0001 C CNN
-	1    6650 4600
-	0    -1   1    0
-$EndComp
-$Comp
-L LFresistor:RESISTOR R10
+P 6650 4450
+F 0 "C7" V 6700 4300 71  0000 R CNN
+F 1 "47 мк 63 В" V 6800 4350 71  0000 R CNN
+F 2 "" H 6650 4450 50  0001 C CNN
+F 3 "" H 6650 4450 50  0001 C CNN
+	1    6650 4450
+	0    -1   1    0
+$EndComp
+$Comp
+L LFresistor:RESISTOR R9
 U 1 1 60358AEB
-P 6650 4150
-F 0 "R10" V 6700 3950 71  0000 R CNN
-F 1 "1 к 1%" V 6800 4050 71  0000 R CNN
-F 2 "IWsmd_case:SMD0805" H 6650 4150 60  0001 C CNN
-F 3 "AmpliOp.sch" V 6898 4072 60  0001 R CNN
-	1    6650 4150
-	0    -1   1    0
-$EndComp
-Wire Wire Line
-	6650 4850 6650 5050
-Text Label 6650 5050 1    50   ~ 0
+P 6650 4000
+F 0 "R9" V 6700 3800 71  0000 R CNN
+F 1 "1 к 1%" V 6800 3900 71  0000 R CNN
+F 2 "IWsmd_case:SMD0805" H 6650 4000 60  0001 C CNN
+F 3 "AmpliOp.sch" V 6898 3922 60  0001 R CNN
+	1    6650 4000
+	0    -1   1    0
+$EndComp
+Wire Wire Line
+	6650 4700 6650 4900
+Text Label 6650 4900 1    50   ~ 0
 GND
 $Comp
@@
 	8300 2400 8300 3400
 $Comp
-L LFresistor:RESISTOR_TRIMMING R12
+L LFresistor:RESISTOR_TRIMMING R11
 U 1 1 60358B03
 P 7650 3800
-F 0 "R12" H 7750 4100 71  0000 C CNN
+F 0 "R11" H 7750 4100 71  0000 C CNN
 F 1 "50 к" H 7750 4000 71  0000 C CNN
 F 2 "IWsmd_case:BOURNS_3224J" H 7650 3800 60  0001 C CNN
@@
 L LFresistor:RESISTOR R4
 U 1 1 60371EE9
-P 3700 4150
-F 0 "R4" V 3750 3950 71  0000 R CNN
-F 1 "1 к 1%" V 3850 4050 71  0000 R CNN
-F 2 "IWsmd_case:SMD0805" H 3700 4150 60  0001 C CNN
-F 3 "AmpliOp.sch" V 3948 4072 60  0001 R CNN
-	1    3700 4150
+P 3700 4000
+F 0 "R4" V 3750 3800 71  0000 R CNN
+F 1 "1 к 1%" V 3850 3900 71  0000 R CNN
+F 2 "IWsmd_case:SMD0805" H 3700 4000 60  0001 C CNN
+F 3 "AmpliOp.sch" V 3948 3922 60  0001 R CNN
+	1    3700 4000
 	0    -1   1    0
 $EndComp
 Connection ~ 3700 3800
 Wire Wire Line
-	3700 3800 3700 4150
-Wire Wire Line
-	3700 4400 3700 4600
+	3700 3800 3700 4000
+Wire Wire Line
+	3700 4250 3700 4450
 $Comp
 L LFbutton:MTS-102-C4-R SB1
@@
 	5350 1950 5350 2400
 $Comp
-L LFbutton:MTS-102-C4-R SB3
+L LFbutton:MTS-102-C4-R SB2
 U 1 1 603D183A
 P 6200 2300
-F 0 "SB3" H 6200 2650 70  0000 C CNN
+F 0 "SB2" H 6200 2650 70  0000 C CNN
 F 1 "MTS-102-C4-R" H 6200 2550 70  0000 C CNN
 F 2 "" V 6150 2200 60  0001 C CNN
@@
 	8300 1950 8300 2400
 $Comp
-L LFresistor:RESISTOR R9
+L LFresistor:RESISTOR R8
 U 1 1 603F3CA4
 P 6550 2500
-F 0 "R9" V 6650 2800 71  0000 R CNN
+F 0 "R8" V 6650 2800 71  0000 R CNN
 F 1 "100 к" V 6750 2900 71  0000 R CNN
 F 2 "IWsmd_case:SMD0805" H 6550 2500 60  0001 C CNN
@@
 	5800 2300 5800 2400
 Wire Wire Line
-	4250 4350 4350 4350
-Wire Wire Line
-	4250 3800 4250 4350
-Wire Wire Line
 	5350 2400 5800 2400
 Wire Wire Line
@@
 	6550 2400 6750 2400
 Wire Wire Line
-	6650 3800 6650 4150
-Wire Wire Line
-	6650 4400 6650 4600
-Text Notes 3550 1650 0    100  ~ 0
-Усилитель на 10, 20 дБ
-Text Notes 6650 1650 0    100  ~ 0
-Усилитель на 20 дБ
+	6650 3800 6650 4000
+Wire Wire Line
+	6650 4250 6650 4450
+Text Notes 3750 1650 0    100  ~ 0
+ Усиление 10 дБ
+Text Notes 6800 1650 0    100  ~ 0
+Усиление 20 дБ
 Text Notes 1050 2240 0    50   ~ 0
 GND
@@
 Text Notes 1000 2440 0    50   ~ 0
 +48 В
-Text Notes 1050 2540 0    50   ~ 0
-GND
 Text Notes 10240 2340 0    50   ~ 0
 GND
@@
 	7200 3800 7650 3800
 $Comp
-L LFresistor:RESISTOR R11
+L LFresistor:RESISTOR R10
 U 1 1 60358961
 P 6950 3800
-F 0 "R11" H 7050 4050 71  0000 C CNN
+F 0 "R10" H 7050 4050 71  0000 C CNN
 F 1 "1 к 1%" H 7100 3950 71  0000 C CNN
 F 2 "IWsmd_case:SMD0805" H 6950 3800 60  0001 C CNN
@@
 	1    0    0    -1
 $EndComp
+Wire Wire Line
+	1650 2200 2000 2200
+Wire Wire Line
+	4250 3800 4700 3800
+Wire Wire Line
+	5100 3800 5350 3800
+Connection ~ 5100 3800
+Wire Wire Line
+	5100 3700 5100 3800
+Wire Wire Line
+	4950 3700 5100 3700
+Wire Wire Line
+	4950 3800 5100 3800
+$Comp
+L LFresistor:RESISTOR_TRIMMING R6
+U 1 1 60388BE5
+P 4700 3800
+F 0 "R6" H 4800 4100 71  0000 C CNN
+F 1 "50 к" H 4800 4000 71  0000 C CNN
+F 2 "IWsmd_case:BOURNS_3224J" H 4700 3800 60  0001 C CNN
+F 3 "AmpliOp.sch" H 4825 4031 60  0001 C CNN
+	1    4700 3800
+	1    0    0    -1
+$EndComp
